Commit message: added parameter for collisionground

File: urdf/niryo_one.urdf_collisionground.xacro (robot description, xacro)
@@ -47,4 +47,10 @@
 	<!-- Links -->
     <link name="ground_link">
+	<collision>
+         <origin xyz="0 0 -0.001" rpy="0 0 0" />
+         <geometry>
+            <box size="1.5 1.5 0.001" />
+         </geometry>
+        </collision>
     </link>
     <link name="base_link">
