Commit message: Added collision box as round link to prevent planning collisions. Rviz visualizes collisions, but move_group still allows to plan

File: urdf/niryo_one.urdf.xacro (robot description, xacro)
@@ -44,8 +44,15 @@
 	<xacro:include filename="$(find niryo_one_description)/urdf/gazebo/niryo_one.transmission.xacro" />
 	<!-- Gripper -->
-	<xacro:include filename="$(find icclab_grasping_niryo)/urdf/niryo_gripper_1.urdf.xacro" />
+	<xacro:include filename="$(find niryo_one_description)/urdf/v2/gripper/niryo_gripper_1.urdf.xacro" />
 	<!--xacro:include filename="$(find niryo_one_description)/urdf/v2/gripper/niryo_gripper_2.urdf.xacro" /-->
 	<!-- Links -->
-    <link name="ground_link"/>
+    <link name="ground_link">
+      <collision>
+         <origin xyz="0 0 0" rpy="0 0 0" />
+         <geometry>
+            <box size="1.5 1.5 0.001" />
+         </geometry>
+       </collision>
+    </link>
     <link name="base_link">
 		<visual>

Commit message: commented collision ground in urdf to use octomap

File: urdf/niryo_one.urdf.xacro (robot description, xacro)
@@ -44,14 +44,14 @@
 	<xacro:include filename="$(find niryo_one_description)/urdf/gazebo/niryo_one.transmission.xacro" />
 	<!-- Gripper -->
-	<xacro:include filename="$(find niryo_one_description)/urdf/v2/gripper/niryo_gripper_1.urdf.xacro" />
+	<xacro:include filename="$(find icclab_grasping_niryo)/urdf/niryo_gripper_1.urdf.xacro" />
 	<!--xacro:include filename="$(find niryo_one_description)/urdf/v2/gripper/niryo_gripper_2.urdf.xacro" /-->
 	<!-- Links -->
     <link name="ground_link">
-      <collision>
+	    <!--  <collision>
          <origin xyz="0 0 0" rpy="0 0 0" />
          <geometry>
             <box size="1.5 1.5 0.001" />
          </geometry>
-       </collision>
+	    </collision> -->
     </link>
     <link name="base_link">

Commit message: path for stl and dae corrected

File: urdf/niryo_one.urdf.xacro (robot description, xacro)
@@ -40,9 +40,10 @@
     <xacro:property name="limit_low_hand_rotation" value="-2.57436" />
     <xacro:property name="limit_up_hand_rotation" value="2.57436" />
-    <xacro:include filename="$(find niryo_one_description)/urdf/gazebo/niryo_one_v2.gazebo.xacro" />
+    <xacro:include filename="$(find niryo_one_description)/urdf/gazebo/niryo_one_v2.urdf.xacro" />
 	<xacro:include filename="$(find niryo_one_description)/urdf/gazebo/utils.xacro" />
 	<xacro:include filename="$(find niryo_one_description)/urdf/gazebo/niryo_one.transmission.xacro" />
 	<!-- Gripper -->
  	<xacro:include filename="$(find niryo_one_description)/urdf/v2/gripper/niryo_gripper_1.urdf.xacro" />
+	<xacro:property name="path" value="/home/ros/catkin_ws/src/niryo_one_ros/niryo_one_description/meshes/v2/" />
 	<!-- Links -->
     <link name="ground_link">
@@ -52,5 +53,5 @@
 			<origin xyz="0 0 0" rpy="0 0 0" />
 			<geometry>
-                <mesh filename="package://niryo_one_description/meshes/v2/collada/base_link.dae" />
+                <mesh filename="${path}/collada/base_link.dae" />
 			</geometry>
         </visual>
@@ -58,5 +59,5 @@
 			<origin xyz="0 0 0" rpy="0 0 0" />
   	   <geometry>
-		        <mesh filename="package://niryo_one_description/meshes/v2/stl/base_link.stl" />
+		        <mesh filename="${path}/stl/base_link.stl" />
             </geometry>
         </collision>
@@ -81,11 +82,11 @@
 			<origin xyz="0 0 0" rpy="0 0 0" />
 			<geometry>
-                <mesh filename="package://niryo_one_description/meshes/v2/collada/shoulder_link.dae" />
-			</geometry>
-		</visual>
-        <collision>
-			<origin xyz="0 0 0" rpy="0 0 0" />
-            <geometry>
-                <mesh filename="package://niryo_one_description/meshes/v2/stl/shoulder_link.stl" />
+                <mesh filename="${path}/collada/shoulder_link.dae" />
+			</geometry>
+		</visual>
+        <collision>
+			<origin xyz="0 0 0" rpy="0 0 0" />
+            <geometry>
+                <mesh filename="${path}/stl/shoulder_link.stl" />
             </geometry>
         </collision>
@@ -103,11 +104,11 @@
 			<origin xyz="0 0 0" rpy="0 0 0" />
 			<geometry>
-                <mesh filename="package://niryo_one_description/meshes/v2/collada/arm_link.dae" />
-			</geometry>
-		</visual>
-        <collision>
-			<origin xyz="0 0 0" rpy="0 0 0" />
-            <geometry>
-                <mesh filename="package://niryo_one_description/meshes/v2/stl/arm_link.stl" />
+                <mesh filename="${path}/collada/arm_link.dae" />
+			</geometry>
+		</visual>
+        <collision>
+			<origin xyz="0 0 0" rpy="0 0 0" />
+            <geometry>
+                <mesh filename="${path}/stl/arm_link.stl" />
             </geometry>
         </collision>
@@ -125,11 +126,11 @@
 			<origin xyz="0 0 0" rpy="0 0 0" />
 			<geometry>
-                <mesh filename="package://niryo_one_description/meshes/v2/collada/elbow_link.dae" />
-			</geometry>
-		</visual>
-        <collision>
-			<origin xyz="0 0 0" rpy="0 0 0" />
-            <geometry>
-                <mesh filename="package://niryo_one_description/meshes/v2/stl/elbow_link.stl" />
+                <mesh filename="${path}/collada/elbow_link.dae" />
+			</geometry>
+		</visual>
+        <collision>
+			<origin xyz="0 0 0" rpy="0 0 0" />
+            <geometry>
+                <mesh filename="${path}/stl/elbow_link.stl" />
             </geometry>
         </collision>
@@ -140,5 +141,5 @@
         		ixx="0.0022" ixy="0.0" ixz="0.0"
         		iyy="0.0" iyz="0.0"
-        		izz="0.022"/>
+        		izz="0.0022"/>
     	</inertial>
 	</link>
@@ -147,11 +148,11 @@
 			<origin xyz="0 0 0" rpy="0 0 0" />
 			<geometry>
-                <mesh filename="package://niryo_one_description/meshes/v2/collada/forearm_link.dae" />
-			</geometry>
-		</visual>
-        <collision>
-			<origin xyz="0 0 0" rpy="0 0 0" />
-            <geometry>
-                <mesh filename="package://niryo_one_description/meshes/v2/stl/forearm_link.stl" />
+                <mesh filename="${path}/collada/forearm_link.dae" />
+			</geometry>
+		</visual>
+        <collision>
+			<origin xyz="0 0 0" rpy="0 0 0" />
+            <geometry>
+                <mesh filename="${path}/stl/forearm_link.stl" />
             </geometry>
         </collision>
@@ -161,5 +162,5 @@
       		<inertia
         		ixx="0.0022" ixy="0.0" ixz="0.0"
-        		iyy="1.0" iyz="0.0"
+        		iyy="0.0" iyz="0.0"
         		izz="0.0022"/>
     	</inertial>
@@ -169,11 +170,11 @@
 			<origin xyz="0 0 0" rpy="0 0 0" />
 			<geometry>
-                <mesh filename="package://niryo_one_description/meshes/v2/collada/wrist_link.dae" />
-			</geometry>
-		</visual>
-        <collision>
-			<origin xyz="0 0 0" rpy="0 0 0" />
-            <geometry>
-                <mesh filename="package://niryo_one_description/meshes/v2/stl/wrist_link.stl" />
+                <mesh filename="${path}/collada/wrist_link.dae" />
+			</geometry>
+		</visual>
+        <collision>
+			<origin xyz="0 0 0" rpy="0 0 0" />
+            <geometry>
+                <mesh filename="${path}/stl/wrist_link.stl" />
             </geometry>
         </collision>
@@ -191,11 +192,11 @@
 			<origin xyz="0 0 0" rpy="0 0 0" />
 			<geometry>
-                <mesh filename="package://niryo_one_description/meshes/v2/collada/hand_link.dae" />
-			</geometry>
-		</visual>
-        <collision>
-			<origin xyz="0 0 0" rpy="0 0 0" />
-            <geometry>
-                <mesh filename="package://niryo_one_description/meshes/v2/stl/hand_link.stl" />
+                <mesh filename="${path}/collada/hand_link.dae" />
+			</geometry>
+		</visual>
+        <collision>
+			<origin xyz="0 0 0" rpy="0 0 0" />
+            <geometry>
+                <mesh filename="${path}/stl/hand_link.stl" />
             </geometry>
         </collision>
@@ -271,5 +272,5 @@
 	</xacro:niryo_gripper_2-->
     <!--plugin-->
-	<gazebo>
+	<!-- <gazebo>
   		<plugin name="gazebo_ros_control" filename="libgazebo_ros_control.so">
       	<robotNamespace></robotNamespace>
@@ -277,4 +278,4 @@
     		<legacyModeNS>true</legacyModeNS>
   		</plugin>
-  	</gazebo>
+  	</gazebo> -->
 </robot>
