Commit message: realsense ported

File: urdf/_d435.gazebo.kinect.xacro (robot description, xacro)
@@ -25,5 +25,5 @@
           </clip>
         </camera>
-        <plugin name="${camera_name}_controller" filename="libgazebo_ros_openni_kinect.so">
+        <!-- <plugin name="${camera_name}_controller" filename="libgazebo_ros_openni_kinect.so">
           <cameraName>${camera_name}</cameraName>
           <alwaysOn>true</alwaysOn>
@@ -31,5 +31,5 @@
           <imageTopicName>color/image_raw</imageTopicName>
           <depthImageTopicName>depth/image_raw</depthImageTopicName>
-          <!-- changed topic to be consistent with what we have on phys robot -->
+          <! changed topic to be consistent with what we have on phys robot
           <pointCloudTopicName>depth_registered/points</pointCloudTopicName>
           <cameraInfoTopicName>color/camera_info</cameraInfoTopicName>
@@ -43,5 +43,5 @@
           <distortion_t2>0.0</distortion_t2>
           <pointCloudCutoff>0.4</pointCloudCutoff>
-        </plugin>
+        </plugin> -->
       </sensor>
     </gazebo>

File: urdf/_d435.urdf.xacro (robot description, xacro)
@@ -28,4 +28,5 @@
     <xacro:property name="d435_cam_depth_py" value="0.0175"/>
     <xacro:property name="d435_cam_depth_pz" value="${d435_cam_height/2}"/>
+    <xacro:property name="path" value="/home/ros/catkin_ws/src/realsense/realsense2_description/meshes/" />
     <material name="${name}_aluminum">
 	  <color rgba="0.5 0.5 0.5 1"/>
@@ -48,5 +49,5 @@
         <geometry>
           <!-- <box size="${d435_cam_width} ${d435_cam_height} ${d435_cam_depth}"/> -->
-          <mesh filename="package://realsense2_description/meshes/d435.dae" />
+          <mesh filename="${path}/d435.dae" />
           <!--<mesh filename="package://realsense2_description/meshes/d435/d435.dae" />-->
         </geometry>
